File: hard/r-2r_dac.sch (KiCad schematic (older format))
At the start: 45 parts, among them J1 Conn_01x04_Male, J2 Conn_01x08_Male, J3 Conn_01x01_Male, J4 Conn_01x01_Male, J5 Conn_01x01_Male, J6 Conn_01x02_Male, Q1 BD135, Q2 BD136, U1 L78L33_TO92, U2 74HC595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

Commit message: in work
Parts:
- added J7, J8, J9: Conn_01x01_Male, Connector_PinHeader_2.54mm:PinHeader_1x01_P2.54mm_Vertical, symbol Connector:Conn_01x01_Male
- added MH1, MH2, MH3, MH4: MountingHole, MountingHole:MountingHole_3.2mm_M3, symbol Mechanical:MountingHole
Connections:
- wire segments 162 -> 167
Changed lines of the file:
@@
 Wire Wire Line
 	7725 4050 7725 4175
-Wire Wire Line
-	6925 3775 6925 4325
-Wire Wire Line
-	6925 4325 6600 4325
-Connection ~ 6600 4325
 $Comp
 L power:GND #PWR015
 U 1 1 5B8297AA
-P 6925 3375
-F 0 "#PWR015" H 6925 3125 50  0001 C CNN
-F 1 "GND" H 6930 3202 50  0000 C CNN
-F 2 "" H 6925 3375 50  0001 C CNN
-F 3 "" H 6925 3375 50  0001 C CNN
-	1    6925 3375
-	-1   0    0    1
-$EndComp
-Wire Wire Line
-	6925 3375 6925 3475
+P 6925 3850
+F 0 "#PWR015" H 6925 3600 50  0001 C CNN
+F 1 "GND" H 6930 3677 50  0000 C CNN
+F 2 "" H 6925 3850 50  0001 C CNN
+F 3 "" H 6925 3850 50  0001 C CNN
+	1    6925 3850
+	1    0    0    -1
+$EndComp
 Wire Wire Line
 	7075 3625 7200 3625
@@
 L power:GND #PWR09
 U 1 1 5B866629
-P 4425 4025
-F 0 "#PWR09" H 4425 3775 50  0001 C CNN
-F 1 "GND" H 4430 3852 50  0000 C CNN
-F 2 "" H 4425 4025 50  0001 C CNN
-F 3 "" H 4425 4025 50  0001 C CNN
-	1    4425 4025
+P 4425 4200
+F 0 "#PWR09" H 4425 3950 50  0001 C CNN
+F 1 "GND" H 4430 4027 50  0000 C CNN
+F 2 "" H 4425 4200 50  0001 C CNN
+F 3 "" H 4425 4200 50  0001 C CNN
+	1    4425 4200
 	1    0    0    -1
 $EndComp
@@
 	4350 3900 4425 3900
 Wire Wire Line
-	4425 3900 4425 4025
+	4425 3900 4425 4050
 $Comp
 L Connector:Conn_01x01_Male J4
@@
 	9625 2300 9625 2400
 NoConn ~ 3800 3850
+$Comp
+L Connector:Conn_01x01_Male J7
+U 1 1 5B84026C
+P 4150 4050
+F 0 "J7" H 4256 4228 50  0000 C CNN
+F 1 "Conn_01x01_Male" H 4256 4137 50  0000 C CNN
+F 2 "Connector_PinHeader_2.54mm:PinHeader_1x01_P2.54mm_Vertical" H 4150 4050 50  0001 C CNN
+F 3 "~" H 4150 4050 50  0001 C CNN
+	1    4150 4050
+	1    0    0    -1
+$EndComp
+Wire Wire Line
+	4350 4050 4425 4050
+Connection ~ 4425 4050
+Wire Wire Line
+	4425 4050 4425 4200
+$Comp
+L Connector:Conn_01x01_Male J8
+U 1 1 5B84F4BB
+P 9825 2025
+F 0 "J8" H 9798 1955 50  0000 R CNN
+F 1 "Conn_01x01_Male" H 9798 2046 50  0000 R CNN
+F 2 "Connector_PinHeader_2.54mm:PinHeader_1x01_P2.54mm_Vertical" H 9825 2025 50  0001 C CNN
+F 3 "~" H 9825 2025 50  0001 C CNN
+	1    9825 2025
+	-1   0    0    1
+$EndComp
+$Comp
+L Connector:Conn_01x01_Male J9
+U 1 1 5B84F531
+P 9825 2200
+F 0 "J9" H 9798 2130 50  0000 R CNN
+F 1 "Conn_01x01_Male" H 9798 2221 50  0000 R CNN
+F 2 "Connector_PinHeader_2.54mm:PinHeader_1x01_P2.54mm_Vertical" H 9825 2200 50  0001 C CNN
+F 3 "~" H 9825 2200 50  0001 C CNN
+	1    9825 2200
+	-1   0    0    1
+$EndComp
+Wire Wire Line
+	9625 2025 9625 1925
+Connection ~ 9625 1925
+Wire Wire Line
+	9625 2200 9625 2300
+Connection ~ 9625 2300
+Wire Wire Line
+	6925 3775 6925 3850
+Wire Wire Line
+	6600 4325 6600 3400
+Wire Wire Line
+	6600 3400 6925 3400
+Wire Wire Line
+	6925 3400 6925 3475
+Connection ~ 6600 4325
+$Comp
+L Mechanical:MountingHole MH1
+U 1 1 5B88AF81
+P 1575 1200
+F 0 "MH1" H 1675 1246 50  0000 L CNN
+F 1 "MountingHole" H 1675 1155 50  0000 L CNN
+F 2 "MountingHole:MountingHole_3.2mm_M3" H 1575 1200 50  0001 C CNN
+F 3 "~" H 1575 1200 50  0001 C CNN
+	1    1575 1200
+	1    0    0    -1
+$EndComp
+$Comp
+L Mechanical:MountingHole MH2
+U 1 1 5B88B072
+P 1600 5100
+F 0 "MH2" H 1700 5146 50  0000 L CNN
+F 1 "MountingHole" H 1700 5055 50  0000 L CNN
+F 2 "MountingHole:MountingHole_3.2mm_M3" H 1600 5100 50  0001 C CNN
+F 3 "~" H 1600 5100 50  0001 C CNN
+	1    1600 5100
+	1    0    0    -1
+$EndComp
+$Comp
+L Mechanical:MountingHole MH4
+U 1 1 5B88B1A1
+P 10275 1200
+F 0 "MH4" H 10375 1246 50  0000 L CNN
+F 1 "MountingHole" H 10375 1155 50  0000 L CNN
+F 2 "MountingHole:MountingHole_3.2mm_M3" H 10275 1200 50  0001 C CNN
+F 3 "~" H 10275 1200 50  0001 C CNN
+	1    10275 1200
+	1    0    0    -1
+$EndComp
+$Comp
+L Mechanical:MountingHole MH3
+U 1 1 5B88B2C4
+P 10250 5525
+F 0 "MH3" H 10350 5571 50  0000 L CNN
+F 1 "MountingHole" H 10350 5480 50  0000 L CNN
+F 2 "MountingHole:MountingHole_3.2mm_M3" H 10250 5525 50  0001 C CNN
+F 3 "~" H 10250 5525 50  0001 C CNN
+	1    10250 5525
+	1    0    0    -1
+$EndComp
 $EndSCHEMATC
