File: hard/r-2r_dac.kicad_pcb (KiCad board)
At the start: 2 copper layers, 109.2 x 58.4 mm, 45 parts, among them J1 Conn_01x04_Male, J2 Conn_01x08_Male, J3 Conn_01x01_Male, J4 Conn_01x01_Male, J5 Conn_01x01_Male, J6 Conn_01x02_Male, Q1 BD135, Q2 BD136, U1 L78L33_TO92, U2 74HC595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

Commit message: in work
Parts:
- added J7: Conn_01x01_Male, Connector_PinHeader_2.54mm:PinHeader_1x01_P2.54mm_Vertical, F.Cu at (138.4, 86.4)
- added J8: Conn_01x01_Male, Connector_PinHeader_2.54mm:PinHeader_1x01_P2.54mm_Vertical, F.Cu at (138.4, 57.1)
- added J9: Conn_01x01_Male, Connector_PinHeader_2.54mm:PinHeader_1x01_P2.54mm_Vertical, F.Cu at (138.4, 88.9)
- added MH1: MountingHole, MountingHole:MountingHole_3.2mm_M3, F.Cu at (57.1, 50.8)
- added MH2: MountingHole, MountingHole:MountingHole_3.2mm_M3, F.Cu at (57.1, 92.7)
- added MH3: MountingHole, MountingHole:MountingHole_3.2mm_M3, F.Cu at (141.0, 50.8)
- added MH4: MountingHole, MountingHole:MountingHole_3.2mm_M3, F.Cu at (141.0, 92.7)
- moved R7 20.7 mm to (69.8, 64.8), turned to 0 degrees
- moved R1 12.7 mm to (61.0, 63.5)
- moved R2 12.7 mm to (61.0, 76.2)
- moved R3 10.5 mm to (63.5, 63.5)
- moved R4 10.5 mm to (63.5, 76.2)
- moved R5 10.5 mm to (66.0, 63.5)
- moved R6 10.5 mm to (66.0, 76.2)
- moved RV1 9.57 mm to (94.0, 52.1), turned to 180 degrees
- moved J1 9.25 mm to (66.0, 59.7), turned to 270 degrees
- moved R26 8.98 mm to (120.7, 54.6)
- moved J6 8.98 mm to (138.4, 80.0)
- moved C4 8.13 mm to (135.9, 72.4)
- moved D1 7.41 mm to (125.7, 72.4)
- moved D2 7.41 mm to (125.7, 83.8)
- moved R10 7.41 mm to (100.6, 83.8)
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Connections:
- RV1 pad 1: GND -> Net-(RV1-Pad1)
- RV1 pad 3: Net-(RV1-Pad3) -> GND
- U3 pad 1: Net-(RV1-Pad3) -> Net-(RV1-Pad1)
- U3 pad 2: Net-(RV1-Pad3) -> Net-(RV1-Pad1)
Routing:
- net VCC: track 5.08 -> 55.7 mm
- net GND: track 91.4 -> 134.0 mm
- net Net-(C4-Pad1): track 12.7 -> 55.3 mm
- net Net-(D1-Pad1): track 3.81 -> 37.7 mm
- net Net-(R1-Pad2): track 0.00 -> 17.6 mm
- net Net-(R3-Pad2): track 0.00 -> 16.5 mm
- net Net-(C3-Pad2): track 0.00 -> 14.7 mm
- net Net-(R7-Pad2): track 0.00 -> 12.5 mm
- net Net-(RV1-Pad1): track 0.00 -> 9.42 mm
- net Net-(R5-Pad2): track 0.00 -> 8.89 mm
- net Net-(J1-Pad3): track 0.00 -> 3.81 mm
- net Net-(J1-Pad2): track 0.00 -> 3.81 mm
- net Net-(J1-Pad1): track 0.00 -> 3.81 mm
- net Net-(C4-Pad2): track 6.35 -> 5.08 mm
- net Net-(D1-Pad2): track 12.5 -> 11.4 mm
Other:
- board size 109.2 x 58.4 mm -> 91.4 x 49.5 mm

Commit message: Last tracks
Parts:
- moved RV1 1.27 mm to (95.2, 52.1)
Routing:
- net GND: track 134.0 -> 246.6 mm
- net Net-(C2-Pad1): track 0.00 -> 57.1 mm
- net VCC: track 55.7 -> 99.2 mm
- net Net-(R15-Pad1): track 3.51 -> 21.3 mm, vias 0 -> 2
- net Net-(RV1-Pad1): track 9.42 -> 8.15 mm
- net Net-(C3-Pad2): track 14.7 -> 13.4 mm
Changed lines of the file:
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@@
     (thickness 1.6)
     (drawings 4)
-    (tracks 146)
+    (tracks 195)
     (zones 0)
     (modules 52)
@@
   )
   (module Potentiometer_THT:Potentiometer_Piher_PT-10-V10_Vertical (layer F.Cu)
-    (at 93.98 52.07 180)
+    (at 95.25 52.07 180)
     (descr "Potentiometer, vertical, Piher PT-10-V10, http://www.piher-nacesa.com/pdf/12-PT10v03.pdf")
     (tags "Potentiometer vertical Piher PT-10-V10")
@@
   (segment (start 135.89 50.8) (end 120.65 50.8) (width 0.8) (layer B.Cu) (net 1))
   (segment (start 120.65 54.61) (end 120.65 50.8) (width 0.8) (layer B.Cu) (net 1))
+  (segment (start 107.95 50.8) (end 107.95 48.26) (width 0.8) (layer B.Cu) (net 1))
+  (segment (start 107.95 48.26) (end 81.28 48.26) (width 0.8) (layer B.Cu) (net 1))
+  (segment (start 81.28 48.26) (end 81.28 52.07) (width 0.8) (layer B.Cu) (net 1))
+  (segment (start 81.28 52.07) (end 78.74 54.61) (width 0.8) (layer B.Cu) (net 1))
+  (segment (start 78.74 54.61) (end 77.47 54.61) (width 0.8) (layer B.Cu) (net 1))
+  (segment (start 76.2 59.69) (end 77.47 58.42) (width 0.8) (layer B.Cu) (net 1))
+  (segment (start 77.47 58.42) (end 77.47 54.61) (width 0.8) (layer B.Cu) (net 1))
   (segment (start 100.33 58.42) (end 100.33 63.5) (width 0.6) (layer B.Cu) (net 2))
   (segment (start 114.3 88.9) (end 120.65 88.9) (width 0.8) (layer B.Cu) (net 2))
@@
   (segment (start 135.89 88.9) (end 135.89 82.55) (width 0.8) (layer B.Cu) (net 2))
   (segment (start 135.89 82.55) (end 135.89 81.28) (width 0.8) (layer B.Cu) (net 2))
-  (segment (start 95.33 58.42) (end 100.33 58.42) (width 0.8) (layer B.Cu) (net 2))
-  (segment (start 93.98 57.07) (end 95.33 58.42) (width 0.8) (layer B.Cu) (net 2))
   (segment (start 72.39 78.74) (end 76.2 78.74) (width 0.8) (layer B.Cu) (net 2))
   (segment (start 76.2 78.74) (end 76.2 69.85) (width 0.8) (layer B.Cu) (net 2))
   (segment (start 76.2 69.85) (end 77.47 68.58) (width 0.8) (layer B.Cu) (net 2))
   (segment (start 77.47 68.58) (end 80.01 68.58) (width 0.8) (layer B.Cu) (net 2))
-  (segment (start 85.09 91.44) (end 114.3 91.44) (width 0.8) (layer B.Cu) (net 2))
   (segment (start 114.3 91.44) (end 114.3 88.9) (width 0.8) (layer B.Cu) (net 2))
   (segment (start 60.96 86.36) (end 63.5 86.36) (width 0.8) (layer B.Cu) (net 2))
@@
   (segment (start 71.12 91.44) (end 72.39 91.44) (width 0.8) (layer B.Cu) (net 2))
   (segment (start 72.39 91.44) (end 85.09 91.44) (width 0.8) (layer B.Cu) (net 2))
-  (segment (start 72.39 49.61) (end 77.47 49.61) (width 0.8) (layer B.Cu) (net 2))
   (segment (start 135.89 81.28) (end 138.43 81.28) (width 0.8) (layer B.Cu) (net 2))
   (segment (start 138.43 81.28) (end 138.43 80.01) (width 0.8) (layer B.Cu) (net 2))
   (segment (start 138.43 88.9) (end 138.43 86.36) (width 0.8) (layer B.Cu) (net 2))
   (segment (start 138.43 88.9) (end 135.89 88.9) (width 0.8) (layer B.Cu) (net 2))
+  (segment (start 74.93 49.61) (end 74.93 59.69) (width 0.8) (layer B.Cu) (net 2))
+  (segment (start 74.93 49.61) (end 77.47 49.61) (width 0.8) (layer B.Cu) (net 2))
+  (segment (start 72.39 49.61) (end 74.93 49.61) (width 0.8) (layer B.Cu) (net 2))
+  (segment (start 74.93 59.69) (end 74.93 62.23) (width 0.8) (layer B.Cu) (net 2))
+  (segment (start 74.93 62.23) (end 82.55 62.23) (width 0.8) (layer B.Cu) (net 2))
+  (segment (start 82.55 62.23) (end 82.55 67.31) (width 0.8) (layer B.Cu) (net 2))
+  (segment (start 82.55 67.31) (end 81.28 68.58) (width 0.8) (layer B.Cu) (net 2))
+  (segment (start 81.28 68.58) (end 80.01 68.58) (width 0.8) (layer B.Cu) (net 2))
+  (segment (start 96.6 58.42) (end 100.33 58.42) (width 0.8) (layer B.Cu) (net 2))
+  (segment (start 95.25 57.07) (end 96.6 58.42) (width 0.8) (layer B.Cu) (net 2))
+  (segment (start 82.55 62.23) (end 82.55 53.34) (width 0.8) (layer B.Cu) (net 2))
+  (segment (start 82.55 53.34) (end 83.82 52.07) (width 0.8) (layer B.Cu) (net 2))
+  (segment (start 83.82 52.07) (end 91.44 52.07) (width 0.8) (layer B.Cu) (net 2))
+  (segment (start 91.44 52.07) (end 91.44 57.15) (width 0.8) (layer B.Cu) (net 2))
+  (segment (start 91.52 57.07) (end 95.25 57.07) (width 0.8) (layer B.Cu) (net 2))
+  (segment (start 91.44 57.15) (end 91.52 57.07) (width 0.8) (layer B.Cu) (net 2))
+  (segment (start 82.55 67.31) (end 93.98 67.31) (width 0.8) (layer B.Cu) (net 2))
+  (segment (start 93.98 67.31) (end 93.98 91.44) (width 0.8) (layer B.Cu) (net 2))
+  (segment (start 85.09 91.44) (end 93.98 91.44) (width 0.8) (layer B.Cu) (net 2))
+  (segment (start 93.98 91.44) (end 114.3 91.44) (width 0.8) (layer B.Cu) (net 2))
+  (segment (start 58.42 59.69) (end 58.42 57.15) (width 0.8) (layer B.Cu) (net 2))
+  (segment (start 58.42 57.15) (end 59.69 55.88) (width 0.8) (layer B.Cu) (net 2))
+  (segment (start 59.69 55.88) (end 67.31 55.88) (width 0.8) (layer B.Cu) (net 2))
+  (segment (start 67.31 55.88) (end 68.58 54.61) (width 0.8) (layer B.Cu) (net 2))
+  (segment (start 68.58 54.61) (end 68.58 49.53) (width 0.8) (layer B.Cu) (net 2))
+  (segment (start 68.66 49.61) (end 72.39 49.61) (width 0.8) (layer B.Cu) (net 2))
+  (segment (start 68.58 49.53) (end 68.66 49.61) (width 0.8) (layer B.Cu) (net 2))
+  (segment (start 72.39 54.61) (end 72.39 58.42) (width 0.8) (layer B.Cu) (net 3))
+  (segment (start 72.39 58.42) (end 73.66 59.69) (width 0.8) (layer B.Cu) (net 3))
+  (segment (start 72.335 59.69) (end 73.66 59.69) (width 0.8) (layer B.Cu) (net 3))
+  (segment (start 69.85 62.175) (end 72.335 59.69) (width 0.8) (layer B.Cu) (net 3))
+  (segment (start 69.85 64.77) (end 69.85 62.175) (width 0.8) (layer B.Cu) (net 3))
+  (segment (start 69.85 64.77) (end 67.31 67.31) (width 0.8) (layer B.Cu) (net 3))
+  (segment (start 67.31 67.31) (end 58.42 67.31) (width 0.8) (layer B.Cu) (net 3))
+  (segment (start 58.42 67.31) (end 58.42 83.82) (width 0.8) (layer B.Cu) (net 3))
+  (segment (start 58.42 83.82) (end 68.58 83.82) (width 0.8) (layer B.Cu) (net 3))
+  (segment (start 68.58 83.82) (end 71.12 86.36) (width 0.8) (layer B.Cu) (net 3))
+  (segment (start 71.12 86.36) (end 72.39 86.36) (width 0.8) (layer B.Cu) (net 3))
   (segment (start 107.95 60.96) (end 110.49 63.5) (width 0.6) (layer B.Cu) (net 4))
   (segment (start 107.95 58.42) (end 107.95 60.96) (width 0.6) (layer B.Cu) (net 4))
@@
   (segment (start 95.25 63.5) (end 97.79 66.04) (width 0.6) (layer B.Cu) (net 4))
   (segment (start 97.79 66.04) (end 107.95 66.04) (width 0.6) (layer B.Cu) (net 4))
-  (segment (start 83.98 54.57) (end 87.59 54.57) (width 0.8) (layer B.Cu) (net 5))
-  (segment (start 87.59 54.57) (end 87.63 54.61) (width 0.8) (layer B.Cu) (net 5))
   (segment (start 87.63 58.38) (end 92.75 63.5) (width 0.8) (layer B.Cu) (net 5))
   (segment (start 87.63 54.61) (end 87.63 58.38) (width 0.8) (layer B.Cu) (net 5))
+  (segment (start 87.59 54.57) (end 87.63 54.61) (width 0.8) (layer B.Cu) (net 5))
+  (segment (start 85.25 54.57) (end 87.59 54.57) (width 0.8) (layer B.Cu) (net 5))
   (segment (start 132.08 69.85) (end 132.08 73.66) (width 0.8) (layer B.Cu) (net 6))
   (segment (start 132.08 73.66) (end 132.08 78.74) (width 0.8) (layer B.Cu) (net 6))
@@
   (segment (start 109.22 71.12) (end 114.3 71.12) (width 0.6) (layer B.Cu) (net 32))
   (segment (start 104.120294 71.139706) (end 104.14 71.12) (width 0.6) (layer B.Cu) (net 33))
-  (segment (start 100.64121 71.139706) (end 104.120294 71.139706) (width 0.6) (layer B.Cu) (net 33))
+  (segment (start 100.33 55.88) (end 102.87 55.88) (width 0.8) (layer B.Cu) (net 33))
+  (segment (start 102.87 55.88) (end 102.87 64.77) (width 0.8) (layer B.Cu) (net 33))
+  (via (at 102.87 64.77) (size 0.8) (drill 0.4) (layers F.Cu B.Cu) (net 33))
+  (segment (start 102.87 71.139706) (end 102.87 67.31) (width 0.6) (layer B.Cu) (net 33))
+  (segment (start 102.87 71.139706) (end 104.120294 71.139706) (width 0.6) (layer B.Cu) (net 33))
+  (segment (start 100.64121 71.139706) (end 102.87 71.139706) (width 0.6) (layer B.Cu) (net 33))
+  (segment (start 102.87 67.31) (end 102.87 67.31) (width 0.8) (layer B.Cu) (net 33))
+  (via (at 102.87 67.31) (size 0.8) (drill 0.4) (layers F.Cu B.Cu) (net 33))
+  (segment (start 102.87 64.77) (end 102.87 67.31) (width 0.8) (layer F.Cu) (net 33))
   (segment (start 100.33 50.8) (end 100.33 53.34) (width 0.8) (layer B.Cu) (net 35))
-  (segment (start 93.98 52.07) (end 95.25 50.8) (width 0.8) (layer B.Cu) (net 35))
-  (segment (start 95.25 50.8) (end 100.33 50.8) (width 0.8) (layer B.Cu) (net 35))
+  (segment (start 100.33 50.8) (end 96.52 50.8) (width 0.8) (layer B.Cu) (net 35))
+  (segment (start 96.52 50.8) (end 95.25 52.07) (width 0.8) (layer B.Cu) (net 35))
 )
